Commit message: feat: add integrated eight-joint state contract

File: ros2_ws/src/tinker_sim_bridge/config/tinker_topic_control.ros2_control.xacro (robot description, xacro)
@@ -22,4 +22,9 @@
       <joint name="joint6"><command_interface name="position"/><command_interface name="velocity"/><state_interface name="position"/><state_interface name="velocity"/><state_interface name="effort"/></joint>
       <joint name="joint7"><command_interface name="position"/><command_interface name="velocity"/><state_interface name="position"/><state_interface name="velocity"/><state_interface name="effort"/></joint>
+      <joint name="drive_joint">
+          <state_interface name="position"/>
+          <state_interface name="velocity"/>
+          <state_interface name="effort"/>
+      </joint>
     </ros2_control>
   </xacro:macro>
